File: pe/Anvita-Yeleswarapu/Anvita-Yeleswarapu.kicad_sch (KiCad schematic)
At the start: 0 parts

Commit message: Update buck converter schematic with initial components
Parts:
- added C? (x2): C, symbol Device:C
- added R? (x2): R, symbol Device:R
- added U?: TPS563208, Package_TO_SOT_SMD:SOT-23-6, symbol Regulator_Switching:TPS563208
